Commit message: Adding updates before trying to pre-train in some manner

File: resources/robots/go1/urdf/go1.urdf (robot description, URDF)
Before this commit: robot go1_description, 23 links, 22 joints
Joints:
- joint FL_calf_joint: limit lower=-2.69653369433 upper=-0.916297857297 effort=33.5 velocity=28 -> lower=-2.721 upper=-0.837 effort=33.5 velocity=28
- joint FL_thigh_joint: limit lower=-1.0471975512 upper=4.18879020479 effort=33.5 velocity=28 -> lower=-0.663 upper=2.966 effort=33.5 velocity=28
- joint FR_calf_joint: limit lower=-2.69653369433 upper=-0.916297857297 effort=33.5 velocity=28 -> lower=-2.721 upper=-0.837 effort=33.5 velocity=28
- joint FR_thigh_joint: limit lower=-1.0471975512 upper=4.18879020479 effort=33.5 velocity=28 -> lower=-0.663 upper=2.966 effort=33.5 velocity=28
- joint RL_calf_joint: limit lower=-2.69653369433 upper=-0.916297857297 effort=33.5 velocity=28 -> lower=-2.721 upper=-0.837 effort=33.5 velocity=28
- joint RL_thigh_joint: limit lower=-1.0471975512 upper=4.18879020479 effort=33.5 velocity=28 -> lower=-0.663 upper=2.966 effort=33.5 velocity=28
- joint RR_calf_joint: limit lower=-2.69653369433 upper=-0.916297857297 effort=33.5 velocity=28 -> lower=-2.721 upper=-0.837 effort=33.5 velocity=28
- joint RR_thigh_joint: limit lower=-1.0471975512 upper=4.18879020479 effort=33.5 velocity=28 -> lower=-0.663 upper=2.966 effort=33.5 velocity=28

Commit message: training model on "hard" dynamics

File: resources/robots/go1/urdf/go1.urdf (robot description, URDF)
Before this commit: robot go1_description, 23 links, 22 joints
Joints:
- joint FL_hip_joint: limit lower=-0.802851455917 upper=0.802851455917 effort=33.5 velocity=50 -> lower=-0.802851455917 upper=0.802851455917 effort=23.7 velocity=50
- joint FL_thigh_joint: limit lower=-0.663 upper=2.966 effort=33.5 velocity=28 -> lower=-0.663 upper=2.966 effort=23.7 velocity=28
- joint FR_hip_joint: limit lower=-0.802851455917 upper=0.802851455917 effort=33.5 velocity=50 -> lower=-0.802851455917 upper=0.802851455917 effort=23.7 velocity=50
- joint FR_thigh_joint: limit lower=-0.663 upper=2.966 effort=33.5 velocity=28 -> lower=-0.663 upper=2.966 effort=23.7 velocity=28
- joint RL_hip_joint: limit lower=-0.802851455917 upper=0.802851455917 effort=33.5 velocity=50 -> lower=-0.802851455917 upper=0.802851455917 effort=23.7 velocity=50
- joint RL_thigh_joint: limit lower=-0.663 upper=2.966 effort=33.5 velocity=28 -> lower=-0.663 upper=2.966 effort=23.7 velocity=28
- joint RR_hip_joint: limit lower=-0.802851455917 upper=0.802851455917 effort=33.5 velocity=50 -> lower=-0.802851455917 upper=0.802851455917 effort=23.7 velocity=50
- joint RR_thigh_joint: limit lower=-0.663 upper=2.966 effort=33.5 velocity=28 -> lower=-0.663 upper=2.966 effort=23.7 velocity=28

Commit message: Minor updates for hard dynamics traning

File: resources/robots/go1/urdf/go1.urdf (robot description, URDF)
Before this commit: robot go1_description, 23 links, 22 joints
Joints:
- joint FL_hip_joint: limit lower=-0.802851455917 upper=0.802851455917 effort=23.7 velocity=50 -> lower=-0.802851455917 upper=0.802851455917 effort=33.5 velocity=50
- joint FL_thigh_joint: limit lower=-0.663 upper=2.966 effort=23.7 velocity=28 -> lower=-0.663 upper=2.966 effort=33.5 velocity=28
- joint FR_hip_joint: limit lower=-0.802851455917 upper=0.802851455917 effort=23.7 velocity=50 -> lower=-0.802851455917 upper=0.802851455917 effort=33.5 velocity=50
- joint FR_thigh_joint: limit lower=-0.663 upper=2.966 effort=23.7 velocity=28 -> lower=-0.663 upper=2.966 effort=33.5 velocity=28
- joint RL_hip_joint: limit lower=-0.802851455917 upper=0.802851455917 effort=23.7 velocity=50 -> lower=-0.802851455917 upper=0.802851455917 effort=33.5 velocity=50
- joint RL_thigh_joint: limit lower=-0.663 upper=2.966 effort=23.7 velocity=28 -> lower=-0.663 upper=2.966 effort=33.5 velocity=28
- joint RR_hip_joint: limit lower=-0.802851455917 upper=0.802851455917 effort=23.7 velocity=50 -> lower=-0.802851455917 upper=0.802851455917 effort=33.5 velocity=50
- joint RR_thigh_joint: limit lower=-0.663 upper=2.966 effort=23.7 velocity=28 -> lower=-0.663 upper=2.966 effort=33.5 velocity=28

Commit message: all last mintue RSS changes. Pushing before splitting off into new repo and updating to most recent genesis_lr repo changes

File: resources/robots/go1/urdf/go1.urdf (robot description, URDF)
Before this commit: robot go1_description, 23 links, 22 joints
Links:
- removed link FL_thigh_shoulder
- removed link FR_thigh_shoulder
- removed link RL_thigh_shoulder
- removed link RR_thigh_shoulder
- added link FL_calf_rotor, mass 0.089; collision cylinder length=0.02 radius=0.035; visual cylinder length=0.02 radius=0.035
- added link FL_hip_rotor, mass 0.089; collision cylinder length=0.02 radius=0.035; visual cylinder length=0.02 radius=0.035
- added link FL_thigh_rotor, mass 0.089; collision cylinder length=0.02 radius=0.035; visual cylinder length=0.02 radius=0.035
- added link FR_calf_rotor, mass 0.089; collision cylinder length=0.02 radius=0.035; visual cylinder length=0.02 radius=0.035
- added link FR_hip_rotor, mass 0.089; collision cylinder length=0.02 radius=0.035; visual cylinder length=0.02 radius=0.035
- added link FR_thigh_rotor, mass 0.089; collision cylinder length=0.02 radius=0.035; visual cylinder length=0.02 radius=0.035
- added link RL_calf_rotor, mass 0.089; collision cylinder length=0.02 radius=0.035; visual cylinder length=0.02 radius=0.035
- added link RL_hip_rotor, mass 0.089; collision cylinder length=0.02 radius=0.035; visual cylinder length=0.02 radius=0.035
- added link RL_thigh_rotor, mass 0.089; collision cylinder length=0.02 radius=0.035; visual cylinder length=0.02 radius=0.035
- added link RR_calf_rotor, mass 0.089; collision cylinder length=0.02 radius=0.035; visual cylinder length=0.02 radius=0.035
- added link RR_hip_rotor, mass 0.089; collision cylinder length=0.02 radius=0.035; visual cylinder length=0.02 radius=0.035
- added link RR_thigh_rotor, mass 0.089; collision cylinder length=0.02 radius=0.035; visual cylinder length=0.02 radius=0.035
- added link camera_chin, mass 1e-5; collision box size=.001 .001 .001; visual mesh filename=package://go1_description/meshes/depthCamera.dae scale=1 1 1
- added link camera_face, mass 1e-5; collision box size=.001 .001 .001; visual mesh filename=package://go1_description/meshes/depthCamera.dae scale=1 1 1
- added link camera_laserscan_link_left
- added link camera_laserscan_link_right
- added link camera_left, mass 1e-5; collision box size=.001 .001 .001; visual mesh filename=package://go1_description/meshes/depthCamera.dae scale=1 1 1
- added link camera_optical_chin
- added link camera_optical_face
- added link camera_optical_left
- added link camera_optical_rearDown
- added link camera_optical_right
- added link camera_rearDown, mass 1e-5; collision box size=.001 .001 .001; visual mesh filename=package://go1_description/meshes/depthCamera.dae scale=1 1 1
- added link camera_right, mass 1e-5; collision box size=.001 .001 .001; visual mesh filename=package://go1_description/meshes/depthCamera.dae scale=1 1 1
- added link ultraSound_face, mass 1e-5; collision box size=.001 .001 .001; visual mesh filename=package://go1_description/meshes/ultraSound.dae scale=1 1 1
- added link ultraSound_left, mass 1e-5; collision box size=.001 .001 .001; visual mesh filename=package://go1_description/meshes/ultraSound.dae scale=1 1 1
- added link ultraSound_right, mass 1e-5; collision box size=.001 .001 .001; visual mesh filename=package://go1_description/meshes/ultraSound.dae scale=1 1 1
- link FL_calf: mass 0.158015 -> 0.135862; geometry collision box size=0.213 0.016 0.016; visual mesh filename=package://go1_description/meshes/calf.dae scale=1 1 1
- link FL_hip: mass 0.510299 -> 0.591; geometry collision cylinder length=0.04 radius=0.046; visual mesh filename=package://go1_description/meshes/hip.dae scale=1 1 1
- link FL_thigh: mass 0.898919 -> 0.92; geometry collision box size=0.213 0.0245 0.034; visual mesh filename=package://go1_description/meshes/thigh.dae scale=1 1 1
- link FR_calf: mass 0.158015 -> 0.135862; geometry collision box size=0.213 0.016 0.016; visual mesh filename=package://go1_description/meshes/calf.dae scale=1 1 1
- link FR_hip: mass 0.510299 -> 0.591; geometry collision cylinder length=0.04 radius=0.046; visual mesh filename=package://go1_description/meshes/hip.dae scale=1 1 1
- link FR_thigh: mass 0.898919 -> 0.92; geometry collision box size=0.213 0.0245 0.034; visual mesh filename=package://go1_description/meshes/thigh_mirror.dae scale=1 1 1
- link RL_calf: mass 0.158015 -> 0.135862; geometry collision box size=0.213 0.016 0.016; visual mesh filename=package://go1_description/meshes/calf.dae scale=1 1 1
- link RL_hip: mass 0.510299 -> 0.591; geometry collision cylinder length=0.04 radius=0.046; visual mesh filename=package://go1_description/meshes/hip.dae scale=1 1 1
- link RL_thigh: mass 0.898919 -> 0.92; geometry collision box size=0.213 0.0245 0.034; visual mesh filename=package://go1_description/meshes/thigh.dae scale=1 1 1
- link RR_calf: mass 0.158015 -> 0.135862; geometry collision box size=0.213 0.016 0.016; visual mesh filename=package://go1_description/meshes/calf.dae scale=1 1 1
- link RR_hip: mass 0.510299 -> 0.591; geometry collision cylinder length=0.04 radius=0.046; visual mesh filename=package://go1_description/meshes/hip.dae scale=1 1 1
- link RR_thigh: mass 0.898919 -> 0.92; geometry collision box size=0.213 0.0245 0.034; visual mesh filename=package://go1_description/meshes/thigh_mirror.dae scale=1 1 1
- link imu_link: geometry collision box size=.001 .001 .001; visual box size=0.001 0.001 0.001
- link trunk: mass 4.8 -> 5.204; geometry collision box size=0.3762 0.0935 0.114; visual mesh filename=package://go1_description/meshes/trunk.dae scale=1 1 1
Joints:
- removed joint FL_hip_fixed
- removed joint FR_hip_fixed
- removed joint RL_hip_fixed
- removed joint RR_hip_fixed
- added joint FL_calf_rotor_joint: type fixed, parent FL_thigh, child FL_calf_rotor, origin xyz=0.0 -0.03235 0 rpy=0 0 0
- added joint FL_hip_rotor_joint: type fixed, parent trunk, child FL_hip_rotor, origin xyz=0.11215 0.04675 0 rpy=0 0 0
- added joint FL_thigh_rotor_joint: type fixed, parent FL_hip, child FL_thigh_rotor, origin xyz=0.0 -0.00015 0 rpy=0 0 0
- added joint FR_calf_rotor_joint: type fixed, parent FR_thigh, child FR_calf_rotor, origin xyz=0.0 0.03235 0 rpy=0 0 0
- added joint FR_hip_rotor_joint: type fixed, parent trunk, child FR_hip_rotor, origin xyz=0.11215 -0.04675 0 rpy=0 0 0
- added joint FR_thigh_rotor_joint: type fixed, parent FR_hip, child FR_thigh_rotor, origin xyz=0.0 0.00015 0 rpy=0 0 0
- added joint RL_calf_rotor_joint: type fixed, parent RL_thigh, child RL_calf_rotor, origin xyz=0.0 -0.03235 0 rpy=0 0 0
- added joint RL_hip_rotor_joint: type fixed, parent trunk, child RL_hip_rotor, origin xyz=-0.11215 0.04675 0 rpy=0 0 0
- added joint RL_thigh_rotor_joint: type fixed, parent RL_hip, child RL_thigh_rotor, origin xyz=0.0 -0.00015 0 rpy=0 0 0
- added joint RR_calf_rotor_joint: type fixed, parent RR_thigh, child RR_calf_rotor, origin xyz=0.0 0.03235 0 rpy=0 0 0
- added joint RR_hip_rotor_joint: type fixed, parent trunk, child RR_hip_rotor, origin xyz=-0.11215 -0.04675 0 rpy=0 0 0
- added joint RR_thigh_rotor_joint: type fixed, parent RR_hip, child RR_thigh_rotor, origin xyz=0.0 0.00015 0 rpy=0 0 0
- added joint camera_joint_chin: type fixed, parent trunk, child camera_chin, origin xyz=0.2522 0.0125 -0.0436 rpy=3.141592653589793 1.5707963267948966 0
- added joint camera_joint_face: type fixed, parent trunk, child camera_face, origin xyz=0.2785 0.0125 0.0167 rpy=3.141592653589793 0 0
- added joint camera_joint_left: type fixed, parent trunk, child camera_left, origin xyz=-0.066 0.082 -0.0176 rpy=3.141592653589793 0.2618 1.5707963267948966
- added joint camera_joint_rearDown: type fixed, parent trunk, child camera_rearDown, origin xyz=-0.0825 0.0125 -0.04365 rpy=3.141592653589793 1.5707963267948966 0
- added joint camera_joint_right: type fixed, parent trunk, child camera_right, origin xyz=-0.041 -0.082 -0.0176 rpy=3.141592653589793 0.2618 -1.5707963267948966
- added joint camera_laserscan_joint_left: type fixed, parent camera_left, child camera_laserscan_link_left, origin xyz=0 0 0 rpy=0 0.2618 0
- added joint camera_laserscan_joint_right: type fixed, parent camera_right, child camera_laserscan_link_right, origin xyz=0 0 0 rpy=0 0.2618 0
- added joint camera_optical_joint_chin: type fixed, parent camera_chin, child camera_optical_chin, origin xyz=0 0 0 rpy=-1.5707963267948966 0 -1.5707963267948966
- added joint camera_optical_joint_face: type fixed, parent camera_face, child camera_optical_face, origin xyz=0 0 0 rpy=-1.5707963267948966 0 -1.5707963267948966
- added joint camera_optical_joint_left: type fixed, parent camera_left, child camera_optical_left, origin xyz=0 0 0 rpy=-1.5707963267948966 0 -1.5707963267948966
- added joint camera_optical_joint_rearDown: type fixed, parent camera_rearDown, child camera_optical_rearDown, origin xyz=0 0 0 rpy=-1.5707963267948966 0 -1.5707963267948966
- added joint camera_optical_joint_right: type fixed, parent camera_right, child camera_optical_right, origin xyz=0 0 0 rpy=-1.5707963267948966 0 -1.5707963267948966
- added joint ultraSound_joint_face: type fixed, parent trunk, child ultraSound_face, origin xyz=0.2747 0.0 -0.0088 rpy=0 0 0
- added joint ultraSound_joint_left: type fixed, parent trunk, child ultraSound_left, origin xyz=-0.0535  0.0826 0.00868 rpy=0 0.2618 1.5707963267948966
- added joint ultraSound_joint_right: type fixed, parent trunk, child ultraSound_right, origin xyz=-0.0535 -0.0826 0.00868 rpy=0 0.2618 -1.5707963267948966
- joint FL_calf_joint: limit lower=-2.721 upper=-0.837 effort=33.5 velocity=28 -> lower=-2.818 upper=-0.888 effort=35.55 velocity=20.06
- joint FL_hip_joint: limit lower=-0.802851455917 upper=0.802851455917 effort=33.5 velocity=50 -> lower=-0.863 upper=0.863 effort=23.7 velocity=30.1
- joint FL_thigh_joint: limit lower=-0.663 upper=2.966 effort=33.5 velocity=28 -> lower=-0.686 upper=4.501 effort=23.7 velocity=30.1
- joint FR_calf_joint: limit lower=-2.721 upper=-0.837 effort=33.5 velocity=28 -> lower=-2.818 upper=-0.888 effort=35.55 velocity=20.06
- joint FR_hip_joint: limit lower=-0.802851455917 upper=0.802851455917 effort=33.5 velocity=50 -> lower=-0.863 upper=0.863 effort=23.7 velocity=30.1
- joint FR_thigh_joint: limit lower=-0.663 upper=2.966 effort=33.5 velocity=28 -> lower=-0.686 upper=4.501 effort=23.7 velocity=30.1
- joint RL_calf_joint: limit lower=-2.721 upper=-0.837 effort=33.5 velocity=28 -> lower=-2.818 upper=-0.888 effort=35.55 velocity=20.06
- joint RL_hip_joint: limit lower=-0.802851455917 upper=0.802851455917 effort=33.5 velocity=50 -> lower=-0.863 upper=0.863 effort=23.7 velocity=30.1
- joint RL_thigh_joint: limit lower=-0.663 upper=2.966 effort=33.5 velocity=28 -> lower=-0.686 upper=4.501 effort=23.7 velocity=30.1
- joint RR_calf_joint: limit lower=-2.721 upper=-0.837 effort=33.5 velocity=28 -> lower=-2.818 upper=-0.888 effort=35.55 velocity=20.06
- joint RR_hip_joint: limit lower=-0.802851455917 upper=0.802851455917 effort=33.5 velocity=50 -> lower=-0.863 upper=0.863 effort=23.7 velocity=30.1
- joint RR_thigh_joint: limit lower=-0.663 upper=2.966 effort=33.5 velocity=28 -> lower=-0.686 upper=4.501 effort=23.7 velocity=30.1
